Commit message: Update nav2.
Signed-off-by: James Goppert <james.goppert@gmail.com>

File: mrbuggy3_description/urdf/mrbuggy3.urdf (robot description, URDF)
Before this commit: robot mrbuggy3, 3 links, 2 joints
Links:
- removed link base_laser
- added link /link/rplidar_link/sensor/rplidar/scan
- added link rplidar_link; visual mesh filename=package://mrbuggy3_description/meshes/rplidar.dae scale=1 1 1
Joints:
- removed joint laser_joint
- added joint rplidar_joint: type fixed, parent base_link, child rplidar_link, origin xyz=0.042 0 0.096 rpy=0 0 0
- added joint rplidar_joint2: type fixed, parent rplidar_link, child /link/rplidar_link/sensor/rplidar/scan, origin xyz=0.0 0.0 0.0 rpy=0 0 0

Commit message: Update launch and urdf.
Signed-off-by: Benjamin Perseghetti <bperseghetti@rudislabs.com>

File: mrbuggy3_description/urdf/mrbuggy3.urdf (robot description, URDF)
Before this commit: robot mrbuggy3, 4 links, 3 joints
Links:
- removed link /link/rplidar_link/sensor/rplidar/scan
- removed link rplidar_link
- added link /link/lidar_link/sensor/lidar/scan
- added link lidar_link; visual mesh filename=package://mrbuggy3_description/meshes/STL27L.dae scale=1 1 1
Joints:
- removed joint rplidar_joint
- removed joint rplidar_joint2
- added joint lidar_joint: type fixed, parent base_link, child lidar_link, origin xyz=0.042 0 0.076 rpy=0 0 0
- added joint lidar_joint2: type fixed, parent lidar_link, child /link/lidar_link/sensor/lidar/scan, origin xyz=0.0 0.0 0.0 rpy=0 0 0

Commit message: Update for real vehicle settings.
Signed-off-by: Benjamin Perseghetti <bperseghetti@rudislabs.com>

File: mrbuggy3_description/urdf/mrbuggy3.urdf (robot description, URDF)
Before this commit: robot mrbuggy3, 4 links, 3 joints
Links:
- removed link /link/lidar_link/sensor/lidar/scan
Joints:
- removed joint lidar_joint2
