Commit message: Updated from mrbuggy3 to second revision b3rb.
Co-authored-by: James Goppert <james.goppert@gmail.com>
Signed-off-by: Benjamin Perseghetti <bperseghetti@rudislabs.com>

File: b3rb_description/urdf/b3rb.urdf (robot description, URDF)
Before this commit: robot mrbuggy3, 3 links, 2 joints
Links:
- link base_link: geometry visual mesh filename=package://b3rb_description/meshes/b3rb.dae scale=1 1 1; visual mesh filename=package://b3rb_description/meshes/wheel.dae scale=1 1 1
- link lidar_link: geometry visual mesh filename=package://b3rb_description/meshes/STL27L.dae scale=1 1 1

Commit message: Update RVIZ model.
Signed-off-by: Benjamin Perseghetti <bperseghetti@rudislabs.com>

File: b3rb_description/urdf/b3rb.urdf (robot description, URDF)
Before this commit: robot b3rb, 3 links, 2 joints
Joints:
- joint lidar_joint: origin xyz=0.042 0 0.076 rpy=0 0 0 -> xyz=0 0 0.155 rpy=0 0 0

Commit message: Add camera to urdf.
Signed-off-by: Benjamin Perseghetti <bperseghetti@rudislabs.com>

File: b3rb_description/urdf/b3rb.urdf (robot description, URDF)
Before this commit: robot b3rb, 3 links, 2 joints
Links:
- added link camera_link
- added link camera_link_optical
Joints:
- added joint camera_joint: type fixed, parent base_link, child camera_link, origin xyz=.189 0 .156 rpy=0 0 0
- added joint camera_optical_joint: type fixed, parent camera_link, child camera_link_optical, origin xyz=0 0 0 rpy=-1.57079632679 0 -1.57079632679

Commit message: Simplify robot rendering.
Signed-off-by: Benjamin Perseghetti <bperseghetti@rudislabs.com>

File: b3rb_description/urdf/b3rb.urdf (robot description, URDF)
Before this commit: robot b3rb, 5 links, 4 joints
Links:
- link camera_link: geometry visual box size=.008 .014 .01; visual box size=.008 .028 .028
- link lidar_link: geometry visual box size=0.039 0.039 0.022; visual cylinder length=0.014 radius=0.018
Joints:
- joint camera_joint: origin xyz=.189 0 .156 rpy=0 0 0 -> xyz=.173 0 .145 rpy=0 0 0
- joint camera_optical_joint: origin xyz=0 0 0 rpy=-1.57079632679 0 -1.57079632679 -> xyz=.016 0 .006 rpy=-1.57079632679 0 -1.57079632679
- joint lidar_joint: origin xyz=0 0 0.155 rpy=0 0 0 -> xyz=0 0 0.191 rpy=0 0 0
